Commit message: Moved files

File: robotlab/urdf/floor.xacro (robot description, xacro)
@@ -2,11 +2,12 @@
 <!--Generates a urdf from the macro in gantry_macro.xacro -->
 <robot name="gantry" xmlns:xacro="http://www.ros.org/wiki/xacro">
-  <xacro:include filename="$(find gantry_support)/urdf/gantry_macro.xacro" />
-  <xacro:gantry prefix=""/>
   <xacro:include filename="$(find kuka_kr16_support)/urdf/kr16_2_macro.xacro" />
-  <xacro:kuka_kr16_2 prefix=""/>
-  <joint name="gantry_robot" type="fixed">
-	<parent link="robot_connection" />
-	<child link="base_link" />
+  <xacro:kuka_kr16_2 prefix="floor_" />
+  <link name="root">
+  </link>
+  <joint name="root_floor" type="fixed">
+	  <origin xyz="0 1 0" rpy="0 0 0"/>
+	  <parent link="root" />
+	  <child link="floor_base_link" />
   </joint>
 </robot>

File: robotlab/urdf/gantry.xacro (robot description, xacro)
@@ -3,10 +3,17 @@
 <robot name="gantry" xmlns:xacro="http://www.ros.org/wiki/xacro">
   <xacro:include filename="$(find gantry_support)/urdf/gantry_macro.xacro" />
-  <xacro:gantry prefix=""/>
+  <xacro:gantry prefix="gantry_"/>
   <xacro:include filename="$(find kuka_kr16_support)/urdf/kr16_2_macro.xacro" />
-  <xacro:kuka_kr16_2 prefix=""/>
+  <xacro:kuka_kr16_2 prefix="gantry_"/>
+  <link name="root">
+  </link>
+  <joint name="root_gantry" type="fixed">
+	  <parent link="root" />
+	  <child link="gantry_root" />
+  </joint>
   <joint name="gantry_robot" type="fixed">
-	<parent link="robot_connection" />
-	<child link="base_link" />
+	  <origin xyz="0 0 0" rpy="0 0 0" />
+	  <parent link="gantry_robot_connection" />
+	  <child link="gantry_base_link" />
   </joint>
 </robot>
