Commit message: Made gazebo macro

File: robotlab/urdf/both_gazebo_macro.xacro (robot description, xacro)
@@ -8,5 +8,5 @@
      <xacro:include filename="$(find gantry_gazebo)/urdf/gazebo.xacro" />
      <xacro:macro name="robotlab_gazebo" params="prefix" >
-	     	<xacro:both prefix="" />
+	     	<xacro:both prefix="${prefix}" />
 		<!-- load transmission file for gantry -->
 		<xacro:gantry_transmission prefix="${prefix}gantry_"/>

File: robotlab/urdf/both_macro.xacro (robot description, xacro)
@@ -11,5 +11,5 @@
 		<link name="${prefix}root">
 		</link>
-		<joint name="${prefix}root_gantry" type="fixed">
+		<joint name="${prefix}root_gantry_wee" type="fixed">
 		        <parent link="${prefix}root" />
 		        <child link="${prefix}gantry_root" />
