Commit message: Corrected rotation of robot base

File: gantry_support/urdf/gantry_robot_macro.xacro (robot description, xacro)
@@ -7,4 +7,5 @@
 	<xacro:kuka_kr16_2 prefix="${prefix}"/>
 	<joint name="${prefix}gantry_robot" type="fixed">
+		<origin xyz="0 0 0" rpy="0 0 ${DEG2RAD * 90}"/>
 		<parent link="${prefix}robot_connection" />
 		<child link="${prefix}base_link" />

File: robotlab/urdf/both_macro.xacro (robot description, xacro)
@@ -4,9 +4,8 @@
 	<xacro:macro name="both" params="prefix">
 		<!-- Load required files -->
-		<xacro:include filename="$(find gantry_support)/urdf/gantry_macro.xacro" />
+		<xacro:include filename="$(find gantry_support)/urdf/gantry_robot_macro.xacro" />
 		<xacro:include filename="$(find kuka_kr16_support)/urdf/kr16_2_macro.xacro" />
 		<!-- Run macros -->
-		<xacro:gantry prefix="${prefix}gantry_"/>
-		<xacro:kuka_kr16_2 prefix="${prefix}gantry_"/>
+		<xacro:gantry_robot prefix="${prefix}gantry_"/>
 		<xacro:kuka_kr16_2 prefix="${prefix}floor_" />
 		<link name="${prefix}root">
@@ -17,13 +16,8 @@
 		</joint>
 		<joint name="${prefix}root_floor" type="fixed">
-		        <origin xyz="0 1 0" rpy="0 0 0"/>
+		        <origin xyz="0 1 0" rpy="0 0 -${KUKA_DEG2RAD * 90}"/>
 		        <parent link="${prefix}root" />
 		        <child link="${prefix}floor_base_link" />
 		</joint>
-		<joint name="${prefix}gantry_robot" type="fixed">
-		        <origin xyz="0 0 0" rpy="0 0 0" />
-		        <parent link="${prefix}gantry_robot_connection" />
-		        <child link="${prefix}gantry_base_link" />
-		</joint>
 	</xacro:macro>
 </robot>
