Commit message: Modified zero position and max velocity in blender

File: gantry_support/urdf/gantry.urdf (robot description, URDF)
Before this commit: robot gantry, 6 links, 5 joints
Joints:
- joint link_arm: limit lower=-0.8 upper=0.8 effort=1.0 velocity=0 -> lower=-1.6 upper=0 effort=1.0 velocity=1.0; origin xyz=-0.164527 0.159154 -0.053205 rpy=1.570796 0 0 -> xyz=-0.164527 -0.651668 -0.053205 rpy=1.570796 0 0
- joint link_leg: axis 0 0 1.0 -> 0 0 -1.0; limit lower=-0.77 upper=0.77 effort=1.0 velocity=0 -> lower=0 upper=1.54 effort=1.0 velocity=1.0; origin xyz=-2.570369 -0.057403 0.034558 rpy=0 0 0 -> xyz=-2.570369 -0.057403 0.844145 rpy=0 0 0
- joint link_trolley: axis 0 0 1.0 -> 0 0 -1.0; limit lower=-2.35 upper=2.35 effort=1.0 velocity=0 -> lower=0 upper=4.7 effort=1.0 velocity=1.0; origin xyz=-1.277963 0.430506 -0.476427 rpy=-1.570796 -1.570796 0 -> xyz=-1.277963 2.407403 -0.476427 rpy=-1.570796 -1.570796 0

File: gantry_support/urdf/gantry_macro.xacro (robot description, xacro)
@@ -58,5 +58,5 @@
       </visual>
       <collision name="${prefix}collision_leg">
-        <origin xyz="0 0.114805 -0.069116" rpy="${DEG2RAD * 90} -${DEG2RAD * 90} 0"/>
+        <origin xyz="0.000315 0.114805 -0.069116" rpy="${DEG2RAD * 90} -${DEG2RAD * 90} 0"/>
         <geometry>
           <mesh filename="package://gantry_support/meshes/VIFS42.000.dae" scale="1.0 1.0 1.0"/>
@@ -89,9 +89,9 @@
     </link>
     <joint name="${prefix}joint_e3" type="prismatic">
-      <origin xyz="-0.164527 0.159154 -0.053205" rpy="${DEG2RAD * 90} 0 0"/>
+      <origin xyz="-0.164527 -0.651668 -0.053205" rpy="${DEG2RAD * 90} 0 0"/>
       <parent link="${prefix}link_trolley"/>
       <child link="${prefix}link_arm"/>
       <axis xyz="0 0 1.0"/>
-      <limit lower="-0.8" upper="0.8" effort="1.0" velocity="100"/>
+      <limit lower="-1.6" upper="0" effort="1.0" velocity="1.0"/>
     </joint>
     <joint name="${prefix}link_base" type="fixed">
@@ -101,16 +101,16 @@
     </joint>
     <joint name="${prefix}joint_e1" type="prismatic">
-      <origin xyz="-2.570369 -0.057403 0.034558" rpy="0 0 0"/>
+      <origin xyz="-2.570369 -0.057403 0.844145" rpy="0 0 0"/>
       <parent link="${prefix}link_base"/>
       <child link="${prefix}link_leg"/>
-      <axis xyz="0 0 1.0"/>
-      <limit lower="-0.77" upper="0.77" effort="1.0" velocity="100"/>
+      <axis xyz="0 0 -1.0"/>
+      <limit lower="0" upper="1.54" effort="1.0" velocity="1.0"/>
     </joint>
     <joint name="${prefix}joint_e2" type="prismatic">
-      <origin xyz="-1.277963 0.430506 -0.476427" rpy="-${DEG2RAD * 90} -${DEG2RAD * 90} 0"/>
+      <origin xyz="-1.277963 2.407403 -0.476427" rpy="-${DEG2RAD * 90} -${DEG2RAD * 90} 0"/>
       <parent link="${prefix}link_leg"/>
       <child link="${prefix}link_trolley"/>
-      <axis xyz="0 0 1.0"/>
-      <limit lower="-2.35" upper="2.35" effort="1.0" velocity="100"/>
+      <axis xyz="0 0 -1.0"/>
+      <limit lower="0" upper="4.7" effort="1.0" velocity="1.0"/>
     </joint>
     <joint name="${prefix}robot_connection" type="fixed">

Commit message: Fixed velocity limits

File: gantry_support/urdf/gantry.urdf (robot description, URDF)
Before this commit: robot gantry, 6 links, 5 joints
Links:
- link link_arm: geometry collision mesh filename=../meshes/Cylinder.stl scale=0.188288 0.188288 0.188288; visual mesh filename=../meshes/VIFS96.stl scale=1.0 1.0 1.0
- link link_base: geometry collision mesh filename=../meshes/VIFS01.000.stl scale=1.0 1.0 1.0; visual mesh filename=../meshes/VIFS01.001.stl scale=1.0 1.0 1.0
- link link_leg: geometry collision mesh filename=../meshes/VIFS42.000.stl scale=1.0 1.0 1.0; visual mesh filename=../meshes/VIFS42.001.stl scale=1.0 1.0 1.0
- link link_trolley: geometry collision mesh filename=../meshes/Cube.005.stl scale=0.129538 0.485533 0.188935; visual mesh filename=../meshes/VIFS43.001.stl scale=1.0 1.0 1.0
Joints:
- joint link_arm: limit lower=-1.6 upper=0 effort=1.0 velocity=1.0 -> lower=-1.6 upper=0 effort=1.0 velocity=0.55
- joint link_trolley: limit lower=0 upper=4.7 effort=1.0 velocity=1.0 -> lower=0 upper=4.7 effort=1.0 velocity=0.83

File: gantry_support/urdf/gantry_macro.xacro (robot description, xacro)
@@ -13,5 +13,5 @@
         <origin xyz="0 0 0" rpy="${DEG2RAD * 90} 0 0"/>
         <geometry>
-          <mesh filename="package://gantry_support/meshes/VIFS96.dae" scale="1.0 1.0 1.0"/>
+          <mesh filename="package://gantry_support/meshes/VIFS96.stl" scale="1.0 1.0 1.0"/>
         </geometry>
         <material name="${prefix}VMtl98"/>
@@ -20,5 +20,5 @@
         <origin xyz="0 0 1.34717" rpy="0 0 0"/>
         <geometry>
-          <mesh filename="package://gantry_support/meshes/Cylinder.dae" scale="0.188288 0.188288 0.188288"/>
+          <mesh filename="package://gantry_support/meshes/Cylinder.stl" scale="0.188288 0.188288 0.188288"/>
         </geometry>
       </collision>
@@ -33,5 +33,5 @@
         <origin xyz="0 0 0" rpy="${DEG2RAD * 90} -${DEG2RAD * 90} 0"/>
         <geometry>
-          <mesh filename="package://gantry_support/meshes/VIFS01.001.dae" scale="1.0 1.0 1.0"/>
+          <mesh filename="package://gantry_support/meshes/VIFS01.001.stl" scale="1.0 1.0 1.0"/>
         </geometry>
         <material name="${prefix}03___Default.001"/>
@@ -40,5 +40,5 @@
         <origin xyz="0 0 0" rpy="${DEG2RAD * 90} -${DEG2RAD * 90} 0"/>
         <geometry>
-          <mesh filename="package://gantry_support/meshes/VIFS01.000.dae" scale="1.0 1.0 1.0"/>
+          <mesh filename="package://gantry_support/meshes/VIFS01.000.stl" scale="1.0 1.0 1.0"/>
         </geometry>
       </collision>
@@ -53,5 +53,5 @@
         <origin xyz="0 0.114805 -0.069116" rpy="${DEG2RAD * 90} -${DEG2RAD * 90} 0"/>
         <geometry>
-          <mesh filename="package://gantry_support/meshes/VIFS42.001.dae" scale="1.0 1.0 1.0"/>
+          <mesh filename="package://gantry_support/meshes/VIFS42.001.stl" scale="1.0 1.0 1.0"/>
         </geometry>
         <material name="${prefix}01___Default.001"/>
@@ -60,5 +60,5 @@
         <origin xyz="0.000315 0.114805 -0.069116" rpy="${DEG2RAD * 90} -${DEG2RAD * 90} 0"/>
         <geometry>
-          <mesh filename="package://gantry_support/meshes/VIFS42.000.dae" scale="1.0 1.0 1.0"/>
+          <mesh filename="package://gantry_support/meshes/VIFS42.000.stl" scale="1.0 1.0 1.0"/>
         </geometry>
       </collision>
@@ -73,5 +73,5 @@
         <origin xyz="0 0 0" rpy="-${DEG2RAD * 180} 0 0"/>
         <geometry>
-          <mesh filename="package://gantry_support/meshes/VIFS43.001.dae" scale="1.0 1.0 1.0"/>
+          <mesh filename="package://gantry_support/meshes/VIFS43.001.stl" scale="1.0 1.0 1.0"/>
         </geometry>
         <material name="${prefix}02___Default.001"/>
@@ -80,5 +80,5 @@
         <origin xyz="-0.020567 0.254046 -0.042038" rpy="${DEG2RAD * 90} 0 0"/>
         <geometry>
-          <mesh filename="package://gantry_support/meshes/Cube.005.dae" scale="0.129538 0.485533 0.188935"/>
+          <mesh filename="package://gantry_support/meshes/Cube.005.stl" scale="0.129538 0.485533 0.188935"/>
         </geometry>
       </collision>
@@ -93,5 +93,5 @@
       <child link="${prefix}link_arm"/>
       <axis xyz="0 0 1.0"/>
-      <limit lower="-1.6" upper="0" effort="1.0" velocity="1.0"/>
+      <limit lower="-1.6" upper="0" effort="1.0" velocity="0.55"/>
     </joint>
     <joint name="${prefix}link_base" type="fixed">
@@ -112,5 +112,5 @@
       <child link="${prefix}link_trolley"/>
       <axis xyz="0 0 -1.0"/>
-      <limit lower="0" upper="4.7" effort="1.0" velocity="1.0"/>
+      <limit lower="0" upper="4.7" effort="1.0" velocity="0.83"/>
     </joint>
     <joint name="${prefix}robot_connection" type="fixed">

Commit message: Joint speed E1

File: gantry_support/urdf/gantry.urdf (robot description, URDF)
Before this commit: robot gantry, 6 links, 5 joints
Links:
- link link_base: mass 100.0 -> None
Joints:
- joint link_leg: limit lower=0 upper=1.54 effort=1.0 velocity=1.0 -> lower=0 upper=1.54 effort=1.0 velocity=0.5

File: gantry_support/urdf/gantry_macro.xacro (robot description, xacro)
@@ -25,9 +25,4 @@
     </link>
     <link name="${prefix}link_base">
-      <inertial>
-        <origin xyz="0 0 0" rpy="0 0 0"/>
-        <mass value="100.0"/>
-        <inertia ixx="71.623734" ixy="3.1e-05" ixz="0" iyy="788.87262" iyz="1.2e-05" izz="851.100647"/>
-      </inertial>
       <visual name="${prefix}visual_base">
         <origin xyz="0 0 0" rpy="${DEG2RAD * 90} -${DEG2RAD * 90} 0"/>
@@ -105,5 +100,5 @@
       <child link="${prefix}link_leg"/>
       <axis xyz="0 0 -1.0"/>
-      <limit lower="0" upper="1.54" effort="1.0" velocity="1.0"/>
+      <limit lower="0" upper="1.54" effort="1.0" velocity="0.5"/>
     </joint>
     <joint name="${prefix}joint_e2" type="prismatic">

File: gantry_support/urdf/gantry_robot.urdf (robot description, URDF)
Before this commit: robot gantry, 15 links, 14 joints
Links:
- link link_base: mass 100.0 -> None
Joints:
- joint joint_e1: limit lower=0 upper=1.54 effort=1.0 velocity=1.0 -> lower=0 upper=1.54 effort=1.0 velocity=0.5

Commit message: Fixed error in export from blender

File: gantry_support/urdf/gantry.urdf (robot description, URDF)
Before this commit: robot gantry, 6 links, 5 joints
Links:
- link link_base: mass None -> 100.0

File: gantry_support/urdf/gantry_macro.xacro (robot description, xacro)
@@ -8,5 +8,5 @@
         <origin xyz="0 0 0" rpy="0 0 0"/>
         <mass value="100.0"/>
-        <inertia ixx="77.157539" ixy="-0.43952" ixz="-0.013708" iyy="77.235046" iyz="-3e-06" izz="1.060431"/>
+        <inertia ixx="77.157539" ixy="-0.43952" ixz="-0.013708" iyy="77.235046" iyz="-8e-06" izz="1.060431"/>
       </inertial>
       <visual name="${prefix}visual_arm">
@@ -25,4 +25,9 @@
     </link>
     <link name="${prefix}link_base">
+      <inertial>
+        <origin xyz="0 0 0" rpy="0 0 0"/>
+        <mass value="100.0"/>
+        <inertia ixx="71.623734" ixy="3.1e-05" ixz="0" iyy="788.87262" iyz="1.2e-05" izz="851.100647"/>
+      </inertial>
       <visual name="${prefix}visual_base">
         <origin xyz="0 0 0" rpy="${DEG2RAD * 90} -${DEG2RAD * 90} 0"/>
@@ -43,5 +48,5 @@
         <origin xyz="0 0.114805 -0.069116" rpy="0 0 0"/>
         <mass value="1000.0"/>
-        <inertia ixx="1880.551147" ixy="0.000265" ixz="0" iyy="7958.77002" iyz="-13.379694" izz="6216.929688"/>
+        <inertia ixx="1880.551147" ixy="0.000232" ixz="0" iyy="7958.77002" iyz="-13.379694" izz="6216.929688"/>
       </inertial>
       <visual name="${prefix}visual_leg">
@@ -63,5 +68,5 @@
         <origin xyz="0 0 0" rpy="0 0 0"/>
         <mass value="100.0"/>
-        <inertia ixx="15.599652" ixy="1.71094" ixz="1.886529" iyy="9.19625" iyz="0.938979" izz="14.022485"/>
+        <inertia ixx="15.599652" ixy="1.71094" ixz="1.886528" iyy="9.19625" iyz="0.938975" izz="14.022485"/>
       </inertial>
       <visual name="${prefix}visual_trolley">

File: gantry_support/urdf/gantry_robot.urdf (robot description, URDF)
Before this commit: robot gantry, 15 links, 14 joints
Links:
- link link_base: mass None -> 100.0
