Commit message: Fixed error in joint link names

File: gantry_support/urdf/gantry_macro.xacro (robot description, xacro)
@@ -90,6 +90,6 @@
     <joint name="${prefix}joint_e3" type="prismatic">
       <origin xyz="-0.164527 0.159154 -0.053205" rpy="${DEG2RAD * 90} 0 0"/>
-      <parent link="link_trolley"/>
-      <child link="link_arm"/>
+      <parent link="${prefix}link_trolley"/>
+      <child link="${prefix}link_arm"/>
       <axis xyz="0 0 1.0"/>
       <limit lower="-0.8" upper="0.8" effort="1.0" velocity="0"/>
@@ -97,11 +97,11 @@
     <joint name="${prefix}link_base" type="fixed">
       <origin xyz="0 0 0" rpy="0 ${DEG2RAD * 90} 0"/>
-      <parent link="root"/>
-      <child link="link_base"/>
+      <parent link="${prefix}root"/>
+      <child link="${prefix}link_base"/>
     </joint>
     <joint name="${prefix}joint_e1" type="prismatic">
       <origin xyz="-2.570369 -0.057403 0.034558" rpy="0 0 0"/>
-      <parent link="link_base"/>
-      <child link="link_leg"/>
+      <parent link="${prefix}link_base"/>
+      <child link="${prefix}link_leg"/>
       <axis xyz="0 0 1.0"/>
       <limit lower="-0.77" upper="0.77" effort="1.0" velocity="0"/>
@@ -109,6 +109,6 @@
     <joint name="${prefix}joint_e2" type="prismatic">
       <origin xyz="-1.277963 0.430506 -0.476427" rpy="-${DEG2RAD * 90} -${DEG2RAD * 90} 0"/>
-      <parent link="link_leg"/>
-      <child link="link_trolley"/>
+      <parent link="${prefix}link_leg"/>
+      <child link="${prefix}link_trolley"/>
       <axis xyz="0 0 1.0"/>
       <limit lower="-2.35" upper="2.35" effort="1.0" velocity="0"/>
@@ -116,6 +116,6 @@
     <joint name="${prefix}robot_connection" type="fixed">
       <origin xyz="-0.026405 0.000343 -1.392678" rpy="-${DEG2RAD * 180} 0 0"/>
-      <parent link="link_arm"/>
-      <child link="robot_connection"/>
+      <parent link="${prefix}link_arm"/>
+      <child link="${prefix}robot_connection"/>
     </joint>
     <material name="${prefix}01___Default.001">

Commit message: Increase speedlimit to avoid division by zero

File: gantry_support/urdf/gantry_macro.xacro (robot description, xacro)
@@ -93,5 +93,5 @@
       <child link="${prefix}link_arm"/>
       <axis xyz="0 0 1.0"/>
-      <limit lower="-0.8" upper="0.8" effort="1.0" velocity="0"/>
+      <limit lower="-0.8" upper="0.8" effort="1.0" velocity="100"/>
     </joint>
     <joint name="${prefix}link_base" type="fixed">
@@ -105,5 +105,5 @@
       <child link="${prefix}link_leg"/>
       <axis xyz="0 0 1.0"/>
-      <limit lower="-0.77" upper="0.77" effort="1.0" velocity="0"/>
+      <limit lower="-0.77" upper="0.77" effort="1.0" velocity="100"/>
     </joint>
     <joint name="${prefix}joint_e2" type="prismatic">
@@ -112,5 +112,5 @@
       <child link="${prefix}link_trolley"/>
       <axis xyz="0 0 1.0"/>
-      <limit lower="-2.35" upper="2.35" effort="1.0" velocity="0"/>
+      <limit lower="-2.35" upper="2.35" effort="1.0" velocity="100"/>
     </joint>
     <joint name="${prefix}robot_connection" type="fixed">

Commit message: link_base that was actually a joint.

File: gantry_support/urdf/gantry_macro.xacro (robot description, xacro)
@@ -95,5 +95,5 @@
       <limit lower="-1.6" upper="0" effort="1.0" velocity="0.55"/>
     </joint>
-    <joint name="${prefix}link_base" type="fixed">
+    <joint name="${prefix}joint_base" type="fixed">
       <origin xyz="0 0 0" rpy="0 ${DEG2RAD * 90} 0"/>
       <parent link="${prefix}root"/>

Commit message: same name on a joint and a link

File: gantry_support/urdf/gantry_macro.xacro (robot description, xacro)
@@ -114,5 +114,5 @@
       <limit lower="0" upper="4.7" effort="1.0" velocity="0.83"/>
     </joint>
-    <joint name="${prefix}robot_connection" type="fixed">
+    <joint name="${prefix}robot_connection_joint" type="fixed">
       <origin xyz="-0.026405 0.000343 -1.392678" rpy="-${DEG2RAD * 180} 0 0"/>
       <parent link="${prefix}link_arm"/>

Commit message: .stl->.dae on the visual meshes. Makes colors work well in gazebo.

File: gantry_support/urdf/gantry_macro.xacro (robot description, xacro)
@@ -13,5 +13,5 @@
         <origin xyz="0 0 0" rpy="${DEG2RAD * 90} 0 0"/>
         <geometry>
-          <mesh filename="package://gantry_support/meshes/VIFS96.stl" scale="1.0 1.0 1.0"/>
+          <mesh filename="package://gantry_support/meshes/VIFS96.dae" scale="1.0 1.0 1.0"/>
         </geometry>
         <material name="${prefix}VMtl98"/>
@@ -33,5 +33,5 @@
         <origin xyz="0 0 0" rpy="${DEG2RAD * 90} -${DEG2RAD * 90} 0"/>
         <geometry>
-          <mesh filename="package://gantry_support/meshes/VIFS01.001.stl" scale="1.0 1.0 1.0"/>
+          <mesh filename="package://gantry_support/meshes/VIFS01.001.dae" scale="1.0 1.0 1.0"/>
         </geometry>
         <material name="${prefix}03___Default.001"/>
@@ -53,5 +53,5 @@
         <origin xyz="0 0.114805 -0.069116" rpy="${DEG2RAD * 90} -${DEG2RAD * 90} 0"/>
         <geometry>
-          <mesh filename="package://gantry_support/meshes/VIFS42.001.stl" scale="1.0 1.0 1.0"/>
+          <mesh filename="package://gantry_support/meshes/VIFS42.001.dae" scale="1.0 1.0 1.0"/>
         </geometry>
         <material name="${prefix}01___Default.001"/>
@@ -73,5 +73,5 @@
         <origin xyz="0 0 0" rpy="-${DEG2RAD * 180} 0 0"/>
         <geometry>
-          <mesh filename="package://gantry_support/meshes/VIFS43.001.stl" scale="1.0 1.0 1.0"/>
+          <mesh filename="package://gantry_support/meshes/VIFS43.001.dae" scale="1.0 1.0 1.0"/>
         </geometry>
         <material name="${prefix}02___Default.001"/>

Commit message: Updated xacro

File: gantry_support/urdf/gantry_macro.xacro (robot description, xacro)
@@ -1,4 +1,4 @@
 <?xml version="1.0"?>
-<robot xmlns:xacro="http://www.ros.org/wiki/xacro">
+<robot xmlns:xacro="http://wiki.ros.org/xacro">
   <xacro:property name="DEG2RAD" value="0.017453292519943295"/>
   <xacro:macro name="gantry" params="prefix">

File: gantry_support/urdf/gantry_robot_macro.xacro (robot description, xacro)
@@ -1,4 +1,4 @@
 <?xml version="1.0"?>
-<robot xmlns:xacro="http://www.ros.org/wiki/xacro">
+<robot xmlns:xacro="http://wiki.ros.org/xacro">
   <xacro:macro name="gantry_robot" params="prefix">
     <xacro:include filename="$(find gantry_support)/urdf/gantry_macro.xacro"/>
@@ -7,5 +7,5 @@
     <xacro:kuka_kr16_2 prefix="${prefix}"/>
     <joint name="${prefix}gantry_robot" type="fixed">
-      <origin xyz="0 0 0" rpy="0 0 ${DEG2RAD * 90}"/>
+      <origin xyz="0 0 0" rpy="0 0 ${radians(90)}"/>
       <parent link="${prefix}robot_connection"/>
       <child link="${prefix}base_link"/>

File: robotlab_support/urdf/robotlab.xacro (robot description, xacro)
@@ -1,5 +1,5 @@
 <?xml version="1.0"?>
 <!--Generates a urdf from the macro in gantry_macro.xacro -->
-<robot xmlns:xacro="http://www.ros.org/wiki/xacro" name="robotlab">
+<robot xmlns:xacro="http://wiki.ros.org/xacro" name="robotlab">
   <xacro:include filename="$(find robotlab_support)/urdf/robotlab_macro.xacro"/>
   <xacro:robotlab prefix=""/>

File: robotlab_support/urdf/robotlab_macro.xacro (robot description, xacro)
@@ -1,5 +1,5 @@
 <?xml version="1.0"?>
 <!--Generates a urdf from the macro in gantry_macro.xacro -->
-<robot xmlns:xacro="http://www.ros.org/wiki/xacro">
+<robot xmlns:xacro="http://wiki.ros.org/xacro">
   <xacro:macro name="robotlab" params="prefix">
     <!-- Load required files -->
@@ -20,5 +20,5 @@
     <xacro:A3_box prefix="${prefix}gantry_"/>
     <link name="${prefix}root">
-		</link>
+    </link>
     <joint name="${prefix}root_gantry" type="fixed">
       <origin xyz="0 0 0.0" rpy="0 0 0"/>
@@ -27,5 +27,5 @@
     </joint>
     <joint name="${prefix}root_floor" type="fixed">
-      <origin xyz="-0.402 0.486 0" rpy="0 0 -${KUKA_DEG2RAD * 90}"/>
+      <origin xyz="-0.402 0.486 0" rpy="0 0 -${radians(90)}"/>
       <parent link="${prefix}root"/>
       <child link="${prefix}floor_base_link"/>
@@ -62,10 +62,10 @@
     </joint>
     <joint name="${prefix}floor_A3_plate_box" type="fixed">
-      <origin xyz="-0.28 0.1 0.18" rpy="0 0 ${KUKA_DEG2RAD * 90}"/>
+      <origin xyz="-0.28 0.1 0.18" rpy="0 0 ${radians(90)}"/>
       <parent link="${prefix}floor_link_3"/>
       <child link="${prefix}floor_A3_box"/>
     </joint>
     <joint name="${prefix}gantry_A3_plate_box" type="fixed">
-      <origin xyz="-0.28 0.1 0.18" rpy="0 0 ${KUKA_DEG2RAD * 90}"/>
+      <origin xyz="-0.28 0.1 0.18" rpy="0 0 ${radians(90)}"/>
       <parent link="${prefix}gantry_link_3"/>
       <child link="${prefix}gantry_A3_box"/>

File: robotlab_support/urdf/schunk_macro.xacro (robot description, xacro)
@@ -1,4 +1,4 @@
 <?xml version="1.0"?>
-<robot xmlns:xacro="http://www.ros.org/wiki/xacro">
+<robot xmlns:xacro="http://wiki.ros.org/xacro">
   <xacro:macro name="FTC-50-80" params="prefix">
     <link name="${prefix}FTC-50-80">

File: robotlab_support/urdf/utility_plate_macro.xacro (robot description, xacro)
@@ -1,4 +1,4 @@
 <?xml version="1.0"?>
-<robot xmlns:xacro="http://www.ros.org/wiki/xacro">
+<robot xmlns:xacro="http://wiki.ros.org/xacro">
   <xacro:macro name="A1_plate" params="prefix">
     <link name="${prefix}A1_utility_plate">
