Commit message: Updated placment with data from SINTEF

File: robotlab_support/urdf/both_macro.xacro (robot description, xacro)
@@ -16,5 +16,5 @@
 		</joint>
 		<joint name="${prefix}root_floor" type="fixed">
-		        <origin xyz="0 1 0" rpy="0 0 -${KUKA_DEG2RAD * 90}"/>
+		        <origin xyz="-0.402 0.486 0" rpy="0 0 -${KUKA_DEG2RAD * 90}"/>
 		        <parent link="${prefix}root" />
 		        <child link="${prefix}floor_base_link" />
