Commit message: Updated with correct speed for E1

File: robotlab_support/urdf/both.urdf (robot description, URDF)
Before this commit: robot robotlab, 25 links, 24 joints
Links:
- link gantry_link_base: mass 100.0 -> None
Joints:
- joint gantry_joint_e1: limit lower=0 upper=1.54 effort=1.0 velocity=1.0 -> lower=0 upper=1.54 effort=1.0 velocity=0.5
