Commit message: Fixed links and joints with the same name.

File: robotlab_support/urdf/robotlab_macro.xacro (robot description, xacro)
@@ -48,10 +48,10 @@
 			<child link="${prefix}floor_A1_utility_plate" />
 		</joint>
-		<joint name="${prefix}floor_A3_box" type="fixed">
+		<joint name="${prefix}floor_A3_plate_box" type="fixed">
 			<origin xyz="-0.28 0.1 0.18" rpy="0 0 ${KUKA_DEG2RAD * 90}"/>
 			<parent link="${prefix}floor_link_3"/>
 			<child link="${prefix}floor_A3_box" />
 		</joint>
-		<joint name="${prefix}gantry_A3_box" type="fixed">
+		<joint name="${prefix}gantry_A3_plate_box" type="fixed">
 			<origin xyz="-0.28 0.1 0.18" rpy="0 0 ${KUKA_DEG2RAD * 90}"/>
 			<parent link="${prefix}gantry_link_3"/>

Commit message: Fixed FTC and SWS macros

File: robotlab_support/urdf/robotlab_macro.xacro (robot description, xacro)
@@ -11,6 +11,8 @@
 		<xacro:gantry_robot prefix="${prefix}gantry_" />
 		<xacro:kuka_kr16_2 prefix="${prefix}floor_" />
-		<xacro:FTC-SWS prefix="${prefix}gantry_" />
-		<xacro:FTC-SWS prefix="${prefix}floor_" />
+		<xacro:FTC-50-80 prefix="${prefix}gantry_" />
+		<xacro:FTC-50-80 prefix="${prefix}floor_" />
+		<xacro:SWK-020 prefix="${prefix}gantry_" />
+		<xacro:SWK-020 prefix="${prefix}floor_" />
 		<xacro:A1_plate prefix="${prefix}gantry_" />
 		<xacro:A1_plate prefix="${prefix}floor_" />
@@ -30,12 +32,22 @@
 		</joint>
 		<joint name="${prefix}gantry_tool0_ftc" type="fixed">
-			<origin xyz="0 0 0" rpy="-${KUKA_DEG2RAD * 90} 0 0"/>
+			<origin xyz="0 0 0" rpy="0 0 0"/>
 			<parent link="${prefix}gantry_tool0" />
-			<child link="${prefix}gantry_FTC-SWS" />
+			<child link="${prefix}gantry_FTC-50-80" />
+		</joint>
+		<joint name="${prefix}gantry_ftc_sws" type="fixed">
+			<origin xyz="0 0 0.0485" rpy="0 0 0"/>
+			<parent link="${prefix}gantry_FTC-50-80" />
+			<child link="${prefix}gantry_SWK-020" />
 		</joint>
 		<joint name="${prefix}floor_tool0_ftc" type="fixed">
-			<origin xyz="0 0 0" rpy="-${KUKA_DEG2RAD * 90} 0 0"/>
+			<origin xyz="0 0 0" rpy="0 0 0"/>
 			<parent link="${prefix}floor_tool0" />
-			<child link="${prefix}floor_FTC-SWS" />
+			<child link="${prefix}floor_FTC-50-80" />
+		</joint>
+		<joint name="${prefix}floor_ftc_sws" type="fixed">
+			<origin xyz="0 0 0.0485" rpy="0 0 0"/>
+			<parent link="${prefix}floor_FTC-50-80" />
+			<child link="${prefix}floor_SWK-020" />
 		</joint>
 		<joint name="${prefix}gantry_A1_utility" type="fixed">

File: robotlab_support/urdf/schunk_macro.xacro (robot description, xacro)
@@ -1,23 +1,22 @@
 <?xml version="1.0"?>
 <robot xmlns:xacro="http://www.ros.org/wiki/xacro">
-	<xacro:macro name="SWK-020" params="prefix">
-		<link name="${prefix}SWK-020" >
-			<visual>
-	        		<origin xyz="0 0 0" rpy="0 0 0"/>
-	        		<geometry>
-			          	<mesh filename="package://robotlab_support/meshes/schunk/visual/SWK-020.stl" scale="0.001 0.001 0.001"/>
-        			</geometry>
-			      	</visual>
-		</link>
-	</xacro:macro>
 	<xacro:macro name="FTC-50-80" params="prefix">
-		<link name="${prefix}ftc" >
-			<visual>
-			<origin xyz="0 0 0" rpy="0 0 0" />
-			<geomentry>
-				<mesh filename="package://robotlab_support/meshes/schunk/visual/FTC-50-80.stl" scale="0.001 0.001 0.001"/>
-			</geomentry>
-			</visual>
-		</link>
+		<link name="${prefix}FTC-50-80" >
+    <visual>
+      <geometry>
+        <cylinder length="0.0485" radius="0.082"/>
+      </geometry>
+    </visual>
+    <collision>
+      <geometry>
+        <cylinder length="0.05" radius="0.1"/>
+      </geometry>
+    </collision>
+    <inertial>
+      <!-- data from http://www.comoso.com/uploads/showcase/manuals/Schunk_Comoso_eng_robot_accessoires.pdf -->
+      <mass value="1.56"/>
+      <inertia ixx="0.00395" ixy="0.0" ixz="0.0" iyy="0.00395" iyz="0.0" izz="0.0058"/>
+    </inertial>
+  </link>
 	</xacro:macro>
 	<xacro:macro name="SWA-020" params="prefix">
@@ -29,28 +28,30 @@
         			</geometry>
 			      	</visual>
+    <inertial>
+      <!-- data from http://www.comoso.com/uploads/showcase/manuals/Schunk_Comoso_eng_robot_accessoires.pdf -->
+      <mass value="0.3"/>
+      <inertia ixx="0.054584" ixy="0.0" ixz="0.0" iyy="0.054584" iyz="0.0" izz="0.10914"/>
+    </inertial>
 		</link>
 	</xacro:macro>
-	<xacro:macro name="FTC-SWS" params="prefix">
-		<link name="${prefix}FTC-SWS" >
-			<intertial>
-				<origin xyz="-0.00141168 -0.03561248 -0.00058552" rpy="0 0 0" />
-				<mass value="2.36" />
-				<inertia ixx="2.6282072064e-6" ixy="-9.42992384e-8" ixz="-5.73180928e-8" iyy="3.8189375488e-6" iyz="-3.91095296e-8" izz="2.7425937408e-6"/>
-			</intertial>
+	<xacro:macro name="SWK-020" params="prefix">
+		<link name="${prefix}SWK-020" >
 			<visual>
-	        		<origin xyz="0 0 0" rpy="0 0 0"/>
+	        		<origin xyz="0 0 0" rpy="${pi/2} ${pi} 0"/>
 	        		<geometry>
-			          	<mesh filename="package://robotlab_support/meshes/schunk/visual/forcetourqe_toolchange.stl" scale="0.04 0.04 0.04"/>
+			          	<mesh filename="package://robotlab_support/meshes/schunk/visual/SWK-020.stl" scale="0.001 0.001 0.001"/>
         			</geometry>
-				<material name="grey">
-				        <color rgba=".2 .2 .2 1"/>
-				</material>
-			</visual>
+			      	</visual>
 			<collision>
-	        		<origin xyz="0 0 0" rpy="0 0 0"/>
+	        		<origin xyz="0 0 0" rpy="${pi/2} ${pi} 0"/>
 	        		<geometry>
-			          	<mesh filename="package://robotlab_support/meshes/schunk/visual/forcetourqe_toolchange.stl" scale="0.05 0.05 0.05"/>
+			          	<mesh filename="package://robotlab_support/meshes/schunk/visual/SWK-020.stl" scale="0.002 0.002 0.002"/>
         			</geometry>
-			</collision>
+			      	</collision>
+    <inertial>
+      <!-- data from http://www.comoso.com/uploads/showcase/manuals/Schunk_Comoso_eng_robot_accessoires.pdf -->
+      <mass value="0.8"/>
+      <inertia ixx="0.14555" ixy="0.0" ixz="0.0" iyy="0.14555" iyz="0.0" izz="0.29104"/>
+    </inertial>
 		</link>
 	</xacro:macro>
