Commit message: Updated moveit config to include robot accessories

File: robotlab_support/urdf/robotlab.urdf (robot description, URDF)
Before this commit: robot robotlab, 25 links, 24 joints
Links:
- added link floor_A1_BOX, mass 0.5; collision box size=0.18 0.12 0.08; visual box size=0.167 0.107 0.065
- added link floor_A1_BOX2, mass 0.5; collision box size=0.18 0.12 0.08; visual box size=0.167 0.107 0.065
- added link floor_A1_DCDC, mass 0.5; collision box size=0.2 0.3 0.15; visual box size=0.17 0.26 0.1
- added link floor_A1_utility_plate, mass 0.5; collision box size=0.7 0.3 0.10; visual box size=0.67 0.26 0.005
- added link floor_A3_box, mass 0.5; collision box size=0.35 0.25 0.1; visual box size=0.28 0.17 0.07
- added link floor_FTC-SWS; collision mesh filename=package://robotlab_support/meshes/schunk/visual/forcetourqe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 scale=0.05 0.05 0.05; visual mesh filename=package://robotlab_support/meshes/schunk/visual/forcetourqe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 scale=0.04 0.04 0.04
- added link gantry_A1_BOX, mass 0.5; collision box size=0.18 0.12 0.08; visual box size=0.167 0.107 0.065
- added link gantry_A1_BOX2, mass 0.5; collision box size=0.18 0.12 0.08; visual box size=0.167 0.107 0.065
- added link gantry_A1_DCDC, mass 0.5; collision box size=0.2 0.3 0.15; visual box size=0.17 0.26 0.1
- added link gantry_A1_utility_plate, mass 0.5; collision box size=0.7 0.3 0.10; visual box size=0.67 0.26 0.005
- added link gantry_A3_box, mass 0.5; collision box size=0.35 0.25 0.1; visual box size=0.28 0.17 0.07
- added link gantry_FTC-SWS; collision mesh filename=package://robotlab_support/meshes/schunk/visual/forcetourqe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 scale=0.05 0.05 0.05; visual mesh filename=package://robotlab_support/meshes/schunk/visual/forcetourqe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 scale=0.04 0.04 0.04
- link gantry_link_base: mass None -> 100.0
Joints:
- removed joint root_gantry_wee
- added joint floor_A1_plate_BOX: type fixed, parent floor_A1_utility_plate, child floor_A1_BOX, origin xyz=-0.168 0.13 -0.0025  rpy=0 0 0
- added joint floor_A1_plate_BOX2: type fixed, parent floor_A1_utility_plate, child floor_A1_BOX2, origin xyz=-0.168 0.13 0.0025  rpy=0 0 0
- added joint floor_A1_plate_DCDC: type fixed, parent floor_A1_utility_plate, child floor_A1_DCDC, origin xyz=0.335 0.13 0.0025 rpy=0 0 0
- added joint floor_A1_utility: type fixed, parent floor_link_1, child floor_A1_utility_plate, origin xyz=0.1 0.30 -0.25 rpy=0 0 0
- added joint floor_A3_box: type fixed, parent floor_link_3, child floor_A3_box, origin xyz=-0.28 0.1 0.18 rpy=0 0 1.57079632679
- added joint floor_tool0_ftc: type fixed, parent floor_tool0, child floor_FTC-SWS, origin xyz=0 0 0 rpy=-1.57079632679 0 0
- added joint gantry_A1_plate_BOX: type fixed, parent gantry_A1_utility_plate, child gantry_A1_BOX, origin xyz=-0.168 0.13 -0.0025  rpy=0 0 0
- added joint gantry_A1_plate_BOX2: type fixed, parent gantry_A1_utility_plate, child gantry_A1_BOX2, origin xyz=-0.168 0.13 0.0025  rpy=0 0 0
- added joint gantry_A1_plate_DCDC: type fixed, parent gantry_A1_utility_plate, child gantry_A1_DCDC, origin xyz=0.335 0.13 0.0025 rpy=0 0 0
- added joint gantry_A1_utility: type fixed, parent gantry_link_1, child gantry_A1_utility_plate, origin xyz=0.1 0.30 -0.25 rpy=0 0 0
- added joint gantry_A3_box: type fixed, parent gantry_link_3, child gantry_A3_box, origin xyz=-0.28 0.1 0.18 rpy=0 0 1.57079632679
- added joint gantry_tool0_ftc: type fixed, parent gantry_tool0, child gantry_FTC-SWS, origin xyz=0 0 0 rpy=-1.57079632679 0 0
- added joint root_gantry_fixed: type fixed, parent root, child gantry_root

Commit message: Regenerated urdf file

File: robotlab_support/urdf/robotlab.urdf (robot description, URDF)
Before this commit: robot robotlab, 37 links, 36 joints
Links:
- removed link floor_FTC-SWS
- removed link gantry_FTC-SWS
- added link floor_FTC-50-80, mass 1.56; collision cylinder length=0.05 radius=0.1; visual cylinder length=0.0485 radius=0.082
- added link floor_SWK-020, mass 0.8; collision mesh filename=package://robotlab_support/meshes/schunk/visual/SWK-020.stl scale=0.002 0.002 0.002; visual mesh filename=package://robotlab_support/meshes/schunk/visual/SWK-020.dae scale=0.001 0.001 0.001
- added link gantry_FTC-50-80, mass 1.56; collision cylinder length=0.05 radius=0.1; visual cylinder length=0.0485 radius=0.082
- added link gantry_SWK-020, mass 0.8; collision mesh filename=package://robotlab_support/meshes/schunk/visual/SWK-020.stl scale=0.002 0.002 0.002; visual mesh filename=package://robotlab_support/meshes/schunk/visual/SWK-020.dae scale=0.001 0.001 0.001
- link gantry_link_arm: geometry collision mesh filename=package://gantry_support/meshes/Cylinder.stl scale=0.188288 0.188288 0.188288; visual mesh filename=package://gantry_support/meshes/VIFS96.dae scale=1.0 1.0 1.0
- link gantry_link_base: geometry collision mesh filename=package://gantry_support/meshes/VIFS01.000.stl scale=1.0 1.0 1.0; visual mesh filename=package://gantry_support/meshes/VIFS01.001.dae scale=1.0 1.0 1.0
- link gantry_link_leg: geometry collision mesh filename=package://gantry_support/meshes/VIFS42.000.stl scale=1.0 1.0 1.0; visual mesh filename=package://gantry_support/meshes/VIFS42.001.dae scale=1.0 1.0 1.0
- link gantry_link_trolley: geometry collision mesh filename=package://gantry_support/meshes/Cube.005.stl scale=0.129538 0.485533 0.188935; visual mesh filename=package://gantry_support/meshes/VIFS43.001.dae scale=1.0 1.0 1.0
Joints:
- removed joint floor_A3_box
- removed joint gantry_A3_box
- removed joint gantry_link_base
- removed joint gantry_robot_connection
- removed joint root_gantry_fixed
- added joint floor_A3_plate_box: type fixed, parent floor_link_3, child floor_A3_box, origin xyz=-0.28 0.1 0.18 rpy=0 0 1.57079632679
- added joint floor_ftc_sws: type fixed, parent floor_FTC-50-80, child floor_SWK-020, origin xyz=0 0 0.0485 rpy=0 0 0
- added joint gantry_A3_plate_box: type fixed, parent gantry_link_3, child gantry_A3_box, origin xyz=-0.28 0.1 0.18 rpy=0 0 1.57079632679
- added joint gantry_ftc_sws: type fixed, parent gantry_FTC-50-80, child gantry_SWK-020, origin xyz=0 0 0.0485 rpy=0 0 0
- added joint gantry_joint_base: type fixed, parent gantry_root, child gantry_link_base, origin xyz=0 0 0 rpy=0 1.57079632679 0
- added joint gantry_robot_connection_joint: type fixed, parent gantry_link_arm, child gantry_robot_connection, origin xyz=-0.026405 0.000343 -1.392678 rpy=-3.14159265359 0 0
- added joint root_gantry: type fixed, parent root, child gantry_root, origin xyz=0 0 0.0 rpy=0 0 0
- joint floor_tool0_ftc: child floor_FTC-SWS -> floor_FTC-50-80; origin xyz=0 0 0 rpy=-1.57079632679 0 0 -> xyz=0 0 0 rpy=0 0 0
- joint gantry_tool0_ftc: child gantry_FTC-SWS -> gantry_FTC-50-80; origin xyz=0 0 0 rpy=-1.57079632679 0 0 -> xyz=0 0 0 rpy=0 0 0
