Commit message: Cleanup

File: gantry_gazebo/urdf/gantry_robot_gazebo_macro.xacro (robot description, xacro)
@@ -24,5 +24,28 @@
       		<child link = "${prefix}root" />
      		<origin xyz="0.0 0.0 0.0" rpy="0.0 0.0 0.0" />
-    	</joint>
+	</joint>
+       <!-- fix for gratvity in KR16 -->
+  <gazebo reference="${prefix}_gantry_base_link">
+    <turnGravityOff>true</turnGravityOff>
+  </gazebo>
+  <gazebo reference="${prefix}_gantry_link_1">
+    <turnGravityOff>true</turnGravityOff>
+  </gazebo>
+  <gazebo reference="${prefix}_gantry_link_2">
+    <turnGravityOff>true</turnGravityOff>
+  </gazebo>
+  <gazebo reference="${prefix}gantry_link_3">
+    <turnGravityOff>true</turnGravityOff>
+  </gazebo>
+  <gazebo reference="${prefix}gantry_link_4">
+    <turnGravityOff>true</turnGravityOff>
+  </gazebo>
+  <gazebo reference="${prefix}gantry_link_5">
+    <turnGravityOff>true</turnGravityOff>
+  </gazebo>
+  <gazebo reference="${prefix}gantry_link_6">
+    <turnGravityOff>true</turnGravityOff>
+  </gazebo>
+ 	<!-- end fix for gravity in kr16 -->
      </xacro:macro>
 </robot>

File: gantry_gazebo/urdf/gantry_transmission_macro.xacro (robot description, xacro)
@@ -34,5 +34,20 @@
                 <mechanicalReduction>1</mechanicalReduction>
             </actuator>
-        </transmission>
+    </transmission>
+    <gazebo reference="${prefix}link_base">
+      <material>Gazebo/Grey</material>
+      <turnGravityOff>true</turnGravityOff>
+    </gazebo>
+    <gazebo reference="${prefix}link_leg">
+      <material>Gazebo/Blue</material>
+      <turnGravityOff>true</turnGravityOff>
+    </gazebo>
+    <gazebo reference="${prefix}link_arm">
+      <material>Gazebo/Blue</material>
+      <turnGravityOff>true</turnGravityOff>
+    </gazebo>
+    <gazebo reference="${prefix}link_trolley">
+      <turnGravityOff>true</turnGravityOff>
+    </gazebo>
     </xacro:macro>
 </robot>

File: robotlab_gazebo/urdf/robotlab_macro.xacro (robot description, xacro)
@@ -12,11 +12,47 @@
     <!-- load floor kr16 transmission -->
     <xacro:kr16_2_transmission prefix="${prefix}floor_" />
-    <!-- ros_control plugin -->
-    <gazebo>
-      <plugin name="gazebo_ros_control" filename="libgazebo_ros_control.so">
-        <robotNamespace>/</robotNamespace>
-        <robotSimType>gazebo_ros_control/DefaultRobotHWSim</robotSimType>
-      </plugin>
-    </gazebo>
+  <gazebo reference="${prefix}gantry_base_link">
+    <turnGravityOff>true</turnGravityOff>
+  </gazebo>
+  <gazebo reference="${prefix}gantry_link_1">
+    <turnGravityOff>true</turnGravityOff>
+  </gazebo>
+  <gazebo reference="${prefix}gantry_link_2">
+    <turnGravityOff>true</turnGravityOff>
+  </gazebo>
+  <gazebo reference="${prefix}gantry_link_3">
+    <turnGravityOff>true</turnGravityOff>
+  </gazebo>
+  <gazebo reference="${prefix}gantry_link_4">
+    <turnGravityOff>true</turnGravityOff>
+  </gazebo>
+  <gazebo reference="${prefix}gantry_link_5">
+    <turnGravityOff>true</turnGravityOff>
+  </gazebo>
+  <gazebo reference="${prefix}gantry_link_6">
+    <turnGravityOff>true</turnGravityOff>
+  </gazebo>
+  <gazebo reference="${prefix}floor_base_link">
+    <turnGravityOff>true</turnGravityOff>
+  </gazebo>
+  <gazebo reference="${prefix}floor_link_1">
+    <turnGravityOff>true</turnGravityOff>
+  </gazebo>
+  <gazebo reference="${prefix}floor_link_2">
+    <turnGravityOff>true</turnGravityOff>
+  </gazebo>
+  <gazebo reference="${prefix}floor_link_3">
+    <turnGravityOff>true</turnGravityOff>
+  </gazebo>
+  <gazebo reference="${prefix}floor_link_4">
+    <turnGravityOff>true</turnGravityOff>
+  </gazebo>
+  <gazebo reference="${prefix}floor_link_5">
+    <turnGravityOff>true</turnGravityOff>
+  </gazebo>
+  <gazebo reference="${prefix}floor_link_6">
+    <turnGravityOff>true</turnGravityOff>
+  </gazebo>
+    <!-- ros_control plugin loaded from kr_16 file-->
   </xacro:macro>
 </robot>

File: robotlab_support/urdf/both.xacro (robot description, xacro)
@@ -2,5 +2,5 @@
 <!--Generates a urdf from the macro in gantry_macro.xacro -->
 <robot name="robotlab" xmlns:xacro="http://www.ros.org/wiki/xacro">
-	<xacro:include filename="$(find robotlab)/urdf/both_macro.xacro" />
+	<xacro:include filename="$(find robotlab_support)/urdf/both_macro.xacro" />
 	<xacro:both prefix="" />
 </robot>
