Commit message: non-transmission related things in the transmission macro.

File: gantry_gazebo/urdf/gantry_transmission_macro.xacro (robot description, xacro)
@@ -35,19 +35,4 @@
             </actuator>
     </transmission>
-    <gazebo reference="${prefix}link_base">
-      <material>Gazebo/Grey</material>
-      <turnGravityOff>true</turnGravityOff>
-    </gazebo>
-    <gazebo reference="${prefix}link_leg">
-      <material>Gazebo/Blue</material>
-      <turnGravityOff>true</turnGravityOff>
-    </gazebo>
-    <gazebo reference="${prefix}link_arm">
-      <material>Gazebo/Blue</material>
-      <turnGravityOff>true</turnGravityOff>
-    </gazebo>
-    <gazebo reference="${prefix}link_trolley">
-      <turnGravityOff>true</turnGravityOff>
-    </gazebo>
     </xacro:macro>
 </robot>
