Commit message: Moved world frame out of macro file

File: gantry_gazebo/urdf/gantry_robot_gazebo.xacro (robot description, xacro)
@@ -4,3 +4,10 @@
     <xacro:include filename="$(find gantry_gazebo)/urdf/gantry_robot_gazebo_macro.xacro" />
     <xacro:gantry_robot_gazebo prefix=""/>
+    <!-- connect gantry to world frame -->
+    <link name="world" />
+    <joint name="world_joint" type="fixed">
+	<parent link="world" />
+	<child link = "root" />
+	<origin xyz="0.0 0.0 0.0" rpy="0.0 0.0 0.0" />
+    </joint>
 </robot>

File: gantry_gazebo/urdf/gantry_robot_gazebo_macro.xacro (robot description, xacro)
@@ -18,11 +18,4 @@
 	    <child link="base_link" />
     	</joint>
-    	<!-- connect gantry to world frame -->
-    	<link name="world" />
-    	<joint name="world_joint" type="fixed">
-    		<parent link="world" />
-      		<child link = "${prefix}root" />
-     		<origin xyz="0.0 0.0 0.0" rpy="0.0 0.0 0.0" />
-	</joint>
        <!-- fix for gratvity in KR16 -->
   <gazebo reference="${prefix}_gantry_base_link">
