Commit message: xmllint formatting

File: gantry_gazebo/urdf/gantry_gazebo.xacro (robot description, xacro)
@@ -1,6 +1,6 @@
 <?xml version="1.0"?>
 <!--Generates a urdf from the macro in gantry_macro.xacro -->
-<robot name="gantry_gazebo" xmlns:xacro="http://www.ros.org/wiki/xacro">
-    <xacro:include filename="$(find gantry_gazebo)/urdf/gantry_gazebo_macro.xacro" />
-    <xacro:gantry_gazebo prefix=""/>
+<robot xmlns:xacro="http://www.ros.org/wiki/xacro" name="gantry_gazebo">
+  <xacro:include filename="$(find gantry_gazebo)/urdf/gantry_gazebo_macro.xacro"/>
+  <xacro:gantry_gazebo prefix=""/>
 </robot>

File: gantry_gazebo/urdf/gantry_gazebo_macro.xacro (robot description, xacro)
@@ -2,15 +2,15 @@
 <!--Generates a urdf from the macro in kr16_2_macro.xacro -->
 <robot xmlns:xacro="http://www.ros.org/wiki/xacro">
-  <xacro:include filename="$(find gantry_support)/urdf/gantry_macro.xacro" />
-  <xacro:include filename="$(find gantry_gazebo)/urdf/gantry_transmission_macro.xacro" />
-  <xacro:include filename="$(find gantry_gazebo)/urdf/gazebo.xacro" />
-  <xacro:macro name="gantry_gazebo" params="prefix" >
+  <xacro:include filename="$(find gantry_support)/urdf/gantry_macro.xacro"/>
+  <xacro:include filename="$(find gantry_gazebo)/urdf/gantry_transmission_macro.xacro"/>
+  <xacro:include filename="$(find gantry_gazebo)/urdf/gazebo.xacro"/>
+  <xacro:macro name="gantry_gazebo" params="prefix">
     <xacro:gantry prefix=""/>
     <xacro:gantry_transmission prefix=""/>
-    <link name="world" />
+    <link name="world"/>
     <joint name="world_joint" type="fixed">
-      <parent link="world" />
-      <child link = "${prefix}root" />
-      <origin xyz="0.0 0.0 0.0" rpy="0.0 0.0 0.0" />
+      <parent link="world"/>
+      <child link="${prefix}root"/>
+      <origin xyz="0.0 0.0 0.0" rpy="0.0 0.0 0.0"/>
     </joint>
   </xacro:macro>

File: gantry_gazebo/urdf/gantry_gravity_macro.xacro (robot description, xacro)
@@ -1,5 +1,5 @@
 <?xml version="1.0"?>
 <robot xmlns:xacro="http://www.ros.org/wiki/xacro">
-<xacro:macro name="gantry_gravity" params="prefix" >
+  <xacro:macro name="gantry_gravity" params="prefix">
     <gazebo reference="${prefix}link_leg">
       <turnGravityOff>true</turnGravityOff>

File: gantry_gazebo/urdf/gantry_robot_gazebo.xacro (robot description, xacro)
@@ -1,13 +1,13 @@
 <?xml version="1.0"?>
 <!--Generates a urdf from the macro in gantry_macro.xacro -->
-<robot name="gantry_robot_gazebo" xmlns:xacro="http://www.ros.org/wiki/xacro">
-    <xacro:include filename="$(find gantry_gazebo)/urdf/gantry_robot_gazebo_macro.xacro" />
-    <xacro:gantry_robot_gazebo prefix=""/>
-    <!-- connect gantry to world frame -->
-    <link name="world" />
-    <joint name="world_joint" type="fixed">
-	<parent link="world" />
-	<child link = "root" />
-	<origin xyz="0.0 0.0 0.0" rpy="0.0 0.0 0.0" />
-    </joint>
+<robot xmlns:xacro="http://www.ros.org/wiki/xacro" name="gantry_robot_gazebo">
+  <xacro:include filename="$(find gantry_gazebo)/urdf/gantry_robot_gazebo_macro.xacro"/>
+  <xacro:gantry_robot_gazebo prefix=""/>
+  <!-- connect gantry to world frame -->
+  <link name="world"/>
+  <joint name="world_joint" type="fixed">
+    <parent link="world"/>
+    <child link="root"/>
+    <origin xyz="0.0 0.0 0.0" rpy="0.0 0.0 0.0"/>
+  </joint>
 </robot>

File: gantry_gazebo/urdf/gantry_robot_gazebo_macro.xacro (robot description, xacro)
@@ -1,44 +1,44 @@
 <?xml version="1.0"?>
 <robot xmlns:xacro="http://www.ros.org/wiki/xacro">
-     <xacro:include filename="$(find gantry_support)/urdf/gantry_macro.xacro" />
-     <xacro:include filename="$(find gantry_gazebo)/urdf/gantry_transmission_macro.xacro" />
-     <xacro:include filename="$(find kuka_kr16_support)/urdf/kr16_2_macro.xacro" />
-     <xacro:include filename="$(find kuka_kr16_gazebo)/urdf/kr16_2_transmission_macro.xacro" />
-     <xacro:include filename="$(find gantry_gazebo)/urdf/gazebo.xacro" />
-     <xacro:macro name="gantry_robot_gazebo" params="prefix" >
-	<!-- load gantry -->
-    	<xacro:gantry prefix=""/>
- 	<xacro:gantry_transmission prefix=""/>
-	<!-- load kr16 -->
-    	<xacro:kuka_kr16_2 prefix=""/>
-    	<xacro:kr16_2_transmission prefix=""/>
-   	<!-- Connect gantry to kr16 -->
-    	<joint name="gantry_robot" type="fixed">
-	    <parent link="robot_connection" />
-	    <child link="base_link" />
-    	</joint>
-       <!-- fix for gratvity in KR16 -->
-  <gazebo reference="${prefix}_gantry_base_link">
-    <turnGravityOff>true</turnGravityOff>
-  </gazebo>
-  <gazebo reference="${prefix}_gantry_link_1">
-    <turnGravityOff>true</turnGravityOff>
-  </gazebo>
-  <gazebo reference="${prefix}_gantry_link_2">
-    <turnGravityOff>true</turnGravityOff>
-  </gazebo>
-  <gazebo reference="${prefix}gantry_link_3">
-    <turnGravityOff>true</turnGravityOff>
-  </gazebo>
-  <gazebo reference="${prefix}gantry_link_4">
-    <turnGravityOff>true</turnGravityOff>
-  </gazebo>
-  <gazebo reference="${prefix}gantry_link_5">
-    <turnGravityOff>true</turnGravityOff>
-  </gazebo>
-  <gazebo reference="${prefix}gantry_link_6">
-    <turnGravityOff>true</turnGravityOff>
-  </gazebo>
- 	<!-- end fix for gravity in kr16 -->
-     </xacro:macro>
+  <xacro:include filename="$(find gantry_support)/urdf/gantry_macro.xacro"/>
+  <xacro:include filename="$(find gantry_gazebo)/urdf/gantry_transmission_macro.xacro"/>
+  <xacro:include filename="$(find kuka_kr16_support)/urdf/kr16_2_macro.xacro"/>
+  <xacro:include filename="$(find kuka_kr16_gazebo)/urdf/kr16_2_transmission_macro.xacro"/>
+  <xacro:include filename="$(find gantry_gazebo)/urdf/gazebo.xacro"/>
+  <xacro:macro name="gantry_robot_gazebo" params="prefix">
+    <!-- load gantry -->
+    <xacro:gantry prefix=""/>
+    <xacro:gantry_transmission prefix=""/>
+    <!-- load kr16 -->
+    <xacro:kuka_kr16_2 prefix=""/>
+    <xacro:kr16_2_transmission prefix=""/>
+    <!-- Connect gantry to kr16 -->
+    <joint name="gantry_robot" type="fixed">
+      <parent link="robot_connection"/>
+      <child link="base_link"/>
+    </joint>
+    <!-- fix for gratvity in KR16 -->
+    <gazebo reference="${prefix}_gantry_base_link">
+      <turnGravityOff>true</turnGravityOff>
+    </gazebo>
+    <gazebo reference="${prefix}_gantry_link_1">
+      <turnGravityOff>true</turnGravityOff>
+    </gazebo>
+    <gazebo reference="${prefix}_gantry_link_2">
+      <turnGravityOff>true</turnGravityOff>
+    </gazebo>
+    <gazebo reference="${prefix}gantry_link_3">
+      <turnGravityOff>true</turnGravityOff>
+    </gazebo>
+    <gazebo reference="${prefix}gantry_link_4">
+      <turnGravityOff>true</turnGravityOff>
+    </gazebo>
+    <gazebo reference="${prefix}gantry_link_5">
+      <turnGravityOff>true</turnGravityOff>
+    </gazebo>
+    <gazebo reference="${prefix}gantry_link_6">
+      <turnGravityOff>true</turnGravityOff>
+    </gazebo>
+    <!-- end fix for gravity in kr16 -->
+  </xacro:macro>
 </robot>

File: gantry_gazebo/urdf/gantry_transmission_macro.xacro (robot description, xacro)
@@ -1,38 +1,38 @@
 <?xml version="1.0"?>
 <robot xmlns:xacro="http://www.ros.org/wiki/xacro">
-    <xacro:macro name="gantry_transmission" params="prefix">
-        <!--joint_e1 transmission-->
-        <transmission name="${prefix}joint_e1_trans">
-            <type>transmission_interface/SimpleTransmission</type>
-            <joint name="${prefix}joint_e1">
-                <hardwareInterface>hardware_interface/PositionJointInterface</hardwareInterface>
-            </joint>
-            <actuator name="${prefix}motor_e1">
-                <hardwareInterface>hardware_interface/PositionJointInterface</hardwareInterface>
-                <mechanicalReduction>1</mechanicalReduction>
-            </actuator>
-        </transmission>
-        <!--joint_e2 transmission-->
-        <transmission name="${prefix}joint_e2_trans">
-            <type>transmission_interface/SimpleTransmission</type>
-            <joint name="${prefix}joint_e2">
-                <hardwareInterface>hardware_interface/PositionJointInterface</hardwareInterface>
-            </joint>
-            <actuator name="${prefix}motor_e2">
-                <hardwareInterface>hardware_interface/PositionJointInterface</hardwareInterface>
-                <mechanicalReduction>1</mechanicalReduction>
-            </actuator>
-        </transmission>
-        <!--joint_e3 transmission-->
-        <transmission name="${prefix}joint_e3_trans">
-            <type>transmission_interface/SimpleTransmission</type>
-            <joint name="${prefix}joint_e3">
-                <hardwareInterface>hardware_interface/PositionJointInterface</hardwareInterface>
-            </joint>
-            <actuator name="${prefix}motor_e3">
-                <hardwareInterface>hardware_interface/PositionJointInterface</hardwareInterface>
-                <mechanicalReduction>1</mechanicalReduction>
-            </actuator>
+  <xacro:macro name="gantry_transmission" params="prefix">
+    <!--joint_e1 transmission-->
+    <transmission name="${prefix}joint_e1_trans">
+      <type>transmission_interface/SimpleTransmission</type>
+      <joint name="${prefix}joint_e1">
+        <hardwareInterface>hardware_interface/PositionJointInterface</hardwareInterface>
+      </joint>
+      <actuator name="${prefix}motor_e1">
+        <hardwareInterface>hardware_interface/PositionJointInterface</hardwareInterface>
+        <mechanicalReduction>1</mechanicalReduction>
+      </actuator>
     </transmission>
-    </xacro:macro>
+    <!--joint_e2 transmission-->
+    <transmission name="${prefix}joint_e2_trans">
+      <type>transmission_interface/SimpleTransmission</type>
+      <joint name="${prefix}joint_e2">
+        <hardwareInterface>hardware_interface/PositionJointInterface</hardwareInterface>
+      </joint>
+      <actuator name="${prefix}motor_e2">
+        <hardwareInterface>hardware_interface/PositionJointInterface</hardwareInterface>
+        <mechanicalReduction>1</mechanicalReduction>
+      </actuator>
+    </transmission>
+    <!--joint_e3 transmission-->
+    <transmission name="${prefix}joint_e3_trans">
+      <type>transmission_interface/SimpleTransmission</type>
+      <joint name="${prefix}joint_e3">
+        <hardwareInterface>hardware_interface/PositionJointInterface</hardwareInterface>
+      </joint>
+      <actuator name="${prefix}motor_e3">
+        <hardwareInterface>hardware_interface/PositionJointInterface</hardwareInterface>
+        <mechanicalReduction>1</mechanicalReduction>
+      </actuator>
+    </transmission>
+  </xacro:macro>
 </robot>

File: gantry_gazebo/urdf/gazebo.xacro (robot description, xacro)
@@ -1,9 +1,9 @@
 <?xml version="1.0"?>
 <robot xmlns:xacro="http://www.ros.org/wiki/xacro">
-    <gazebo>
-        <plugin name="ros_control" filename="libgazebo_ros_control.so">
-            <!--<robotNamespace>/</robotNamespace>-->
-            <!--<robotSimType>gazebo_ros_control/DefaultRobotHWSim</robotSimType>-->
-        </plugin>
-    </gazebo>
+  <gazebo>
+    <plugin name="ros_control" filename="libgazebo_ros_control.so">
+      <!--<robotNamespace>/</robotNamespace>-->
+      <!--<robotSimType>gazebo_ros_control/DefaultRobotHWSim</robotSimType>-->
+    </plugin>
+  </gazebo>
 </robot>

File: gantry_support/urdf/gantry.xacro (robot description, xacro)
@@ -1,6 +1,6 @@
 <?xml version="1.0"?>
 <!--Generates a urdf from the macro in gantry_macro.xacro -->
-<robot name="gantry" xmlns:xacro="http://www.ros.org/wiki/xacro">
-  <xacro:include filename="$(find gantry_support)/urdf/gantry_macro.xacro" />
+<robot xmlns:xacro="http://www.ros.org/wiki/xacro" name="gantry">
+  <xacro:include filename="$(find gantry_support)/urdf/gantry_macro.xacro"/>
   <xacro:gantry prefix=""/>
 </robot>

File: gantry_support/urdf/gantry_macro.xacro (robot description, xacro)
@@ -1,7 +1,7 @@
 <?xml version="1.0"?>
 <robot xmlns:xacro="http://www.ros.org/wiki/xacro">
-<xacro:property name="DEG2RAD" value="0.017453292519943295"/>
-<xacro:macro name="gantry" params="prefix">
-<!-- created with Phobos 0.7 -->
+  <xacro:property name="DEG2RAD" value="0.017453292519943295"/>
+  <xacro:macro name="gantry" params="prefix">
+    <!-- created with Phobos 0.7 -->
     <link name="${prefix}link_arm">
       <inertial>

File: gantry_support/urdf/gantry_robot.xacro (robot description, xacro)
@@ -1,6 +1,6 @@
 <?xml version="1.0"?>
 <!--Generates a urdf from the macro in gantry_macro.xacro -->
-<robot name="gantry" xmlns:xacro="http://www.ros.org/wiki/xacro">
-	<xacro:include filename="$(find gantry_support)/urdf/gantry_robot_macro.xacro" />
-	<xacro:gantry_robot prefix="" />
+<robot xmlns:xacro="http://www.ros.org/wiki/xacro" name="gantry">
+  <xacro:include filename="$(find gantry_support)/urdf/gantry_robot_macro.xacro"/>
+  <xacro:gantry_robot prefix=""/>
 </robot>

File: gantry_support/urdf/gantry_robot_macro.xacro (robot description, xacro)
@@ -1,14 +1,14 @@
 <?xml version="1.0"?>
 <robot xmlns:xacro="http://www.ros.org/wiki/xacro">
-<xacro:macro name="gantry_robot" params="prefix">
-	<xacro:include filename="$(find gantry_support)/urdf/gantry_macro.xacro" />
-	<xacro:include filename="$(find kuka_kr16_support)/urdf/kr16_2_macro.xacro" />
-	<xacro:gantry prefix="${prefix}"/>
-	<xacro:kuka_kr16_2 prefix="${prefix}"/>
-	<joint name="${prefix}gantry_robot" type="fixed">
-		<origin xyz="0 0 0" rpy="0 0 ${DEG2RAD * 90}"/>
-		<parent link="${prefix}robot_connection" />
-		<child link="${prefix}base_link" />
-  	</joint>
-</xacro:macro>
+  <xacro:macro name="gantry_robot" params="prefix">
+    <xacro:include filename="$(find gantry_support)/urdf/gantry_macro.xacro"/>
+    <xacro:include filename="$(find kuka_kr16_support)/urdf/kr16_2_macro.xacro"/>
+    <xacro:gantry prefix="${prefix}"/>
+    <xacro:kuka_kr16_2 prefix="${prefix}"/>
+    <joint name="${prefix}gantry_robot" type="fixed">
+      <origin xyz="0 0 0" rpy="0 0 ${DEG2RAD * 90}"/>
+      <parent link="${prefix}robot_connection"/>
+      <child link="${prefix}base_link"/>
+    </joint>
+  </xacro:macro>
 </robot>

File: robotlab_gazebo/urdf/gazebo.xacro (robot description, xacro)
@@ -1,8 +1,8 @@
 <?xml version="1.0"?>
 <robot xmlns:xacro="http://www.ros.org/wiki/xacro">
-    <gazebo>
-      <plugin name="ros_control" filename="libgazebo_ros_control.so">
-	<!-- This plugin is required to link up gazebo and ros control. -->
-      </plugin>
-    </gazebo>
+  <gazebo>
+    <plugin name="ros_control" filename="libgazebo_ros_control.so">
+      <!-- This plugin is required to link up gazebo and ros control. -->
+    </plugin>
+  </gazebo>
 </robot>

File: robotlab_gazebo/urdf/robotlab.xacro (robot description, xacro)
@@ -1,4 +1,4 @@
-<?xml version="1.0" ?>
-<robot name="robotlab" xmlns:xacro="http://www.ros.org/wiki/xacro">
+<?xml version="1.0"?>
+<robot xmlns:xacro="http://www.ros.org/wiki/xacro" name="robotlab">
   <xacro:include filename="$(find robotlab_gazebo)/urdf/robotlab_macro.xacro"/>
   <xacro:robotlab_gazebo prefix=""/>
@@ -8,5 +8,5 @@
     <parent link="world"/>
     <child link="root"/>
-    <origin xyz="0.0 0.0 0.015" rpy="0.0 0.0 0.0" />
+    <origin xyz="0.0 0.0 0.015" rpy="0.0 0.0 0.0"/>
   </joint>
 </robot>

File: robotlab_gazebo/urdf/robotlab_macro.xacro (robot description, xacro)
@@ -10,29 +10,29 @@
   <xacro:include filename="$(find robotlab_gazebo)/urdf/gazebo.xacro"/>
   <!-- Load gravity config for gantry and KR16 -->
-  <xacro:include filename="$(find gantry_gazebo)/urdf/gantry_gravity_macro.xacro" />
-  <xacro:include filename="$(find kuka_kr16_gazebo)/urdf/kr16_2_gravity_macro.xacro" />
+  <xacro:include filename="$(find gantry_gazebo)/urdf/gantry_gravity_macro.xacro"/>
+  <xacro:include filename="$(find kuka_kr16_gazebo)/urdf/kr16_2_gravity_macro.xacro"/>
   <!-- Load colors for utility plates -->
-  <xacro:include filename="$(find robotlab_gazebo)/urdf/utility_plate_gazebo_macro.xacro" />
+  <xacro:include filename="$(find robotlab_gazebo)/urdf/utility_plate_gazebo_macro.xacro"/>
   <!-- Done loading macros -->
   <!-- Make the Gazebo version of the robotlab macro  -->
-  <xacro:macro name="robotlab_gazebo" params="prefix" >
+  <xacro:macro name="robotlab_gazebo" params="prefix">
     <!-- load robots -->
-    <xacro:robotlab prefix="${prefix}" />
+    <xacro:robotlab prefix="${prefix}"/>
     <!-- Utility plate colors -->
-    <xacro:A1_plate_gazebo prefix="${prefix}gantry_" />
-    <xacro:A3_box_gazebo prefix="${prefix}gantry_" />
-    <xacro:A1_plate_gazebo prefix="${prefix}floor_" />
-    <xacro:A3_box_gazebo prefix="${prefix}floor_" />
+    <xacro:A1_plate_gazebo prefix="${prefix}gantry_"/>
+    <xacro:A3_box_gazebo prefix="${prefix}gantry_"/>
+    <xacro:A1_plate_gazebo prefix="${prefix}floor_"/>
+    <xacro:A3_box_gazebo prefix="${prefix}floor_"/>
     <!-- load transmission files for gantry and KR16 -->
-    <xacro:gantry_transmission prefix="${prefix}gantry_" />
-    <xacro:kr16_2_transmission prefix="${prefix}gantry_" />
-    <xacro:kr16_2_transmission prefix="${prefix}floor_" />
+    <xacro:gantry_transmission prefix="${prefix}gantry_"/>
+    <xacro:kr16_2_transmission prefix="${prefix}gantry_"/>
+    <xacro:kr16_2_transmission prefix="${prefix}floor_"/>
     <!-- Load gravity settings -->
     <!-- The robots only have position control. It compensates for gravity using servo and breaks -->
-    <xacro:gantry_gravity prefix="${prefix}gantry_" />
-    <xacro:kr16_2_gravity prefix="${prefix}gantry_" />
-    <xacro:kr16_2_gravity prefix="${prefix}floor_" />
+    <xacro:gantry_gravity prefix="${prefix}gantry_"/>
+    <xacro:kr16_2_gravity prefix="${prefix}gantry_"/>
+    <xacro:kr16_2_gravity prefix="${prefix}floor_"/>
     <gazebo reference="${prefix}root">
-	<static>true</static>
+      <static>true</static>
     </gazebo>
     <!-- ros_control plugin loaded from kr_16 file-->

File: robotlab_gazebo/urdf/utility_plate_gazebo_macro.xacro (robot description, xacro)
@@ -1,27 +1,27 @@
 <?xml version="1.0"?>
 <robot xmlns:xacro="http://www.ros.org/wiki/xacro">
-	<xacro:macro name="A1_plate_gazebo" params="prefix">
-		<gazebo reference="${prefix}A1_utility_plate">
-			<turnGravityOff>true</turnGravityOff>
-			 <material>Gazebo/FlatBlack</material>
-		</gazebo>
-		<gazebo reference="${prefix}A1_BOX">
-			 <material>Gazebo/FlatBlack</material>
-			<turnGravityOff>true</turnGravityOff>
-		</gazebo>
-		<gazebo reference="${prefix}A1_BOX2">
-			 <material>Gazebo/FlatBlack</material>
-			<turnGravityOff>true</turnGravityOff>
-		</gazebo>
-		<gazebo reference="${prefix}A1_DCDC">
-			 <material>Gazebo/Grey</material>
-			<turnGravityOff>true</turnGravityOff>
-		</gazebo>
-	</xacro:macro>
-	<xacro:macro name="A3_box_gazebo" params="prefix">
-		<gazebo reference="${prefix}A3_box">
-			 <material>Gazebo/LightGrey</material>
-			<turnGravityOff>true</turnGravityOff>
-		</gazebo>
-	</xacro:macro>
+  <xacro:macro name="A1_plate_gazebo" params="prefix">
+    <gazebo reference="${prefix}A1_utility_plate">
+      <turnGravityOff>true</turnGravityOff>
+      <material>Gazebo/FlatBlack</material>
+    </gazebo>
+    <gazebo reference="${prefix}A1_BOX">
+      <material>Gazebo/FlatBlack</material>
+      <turnGravityOff>true</turnGravityOff>
+    </gazebo>
+    <gazebo reference="${prefix}A1_BOX2">
+      <material>Gazebo/FlatBlack</material>
+      <turnGravityOff>true</turnGravityOff>
+    </gazebo>
+    <gazebo reference="${prefix}A1_DCDC">
+      <material>Gazebo/Grey</material>
+      <turnGravityOff>true</turnGravityOff>
+    </gazebo>
+  </xacro:macro>
+  <xacro:macro name="A3_box_gazebo" params="prefix">
+    <gazebo reference="${prefix}A3_box">
+      <material>Gazebo/LightGrey</material>
+      <turnGravityOff>true</turnGravityOff>
+    </gazebo>
+  </xacro:macro>
 </robot>

File: robotlab_support/urdf/floor.xacro (robot description, xacro)
@@ -1,13 +1,13 @@
 <?xml version="1.0"?>
 <!--Generates a urdf from the macro in gantry_macro.xacro -->
-<robot name="gantry" xmlns:xacro="http://www.ros.org/wiki/xacro">
-  <xacro:include filename="$(find kuka_kr16_support)/urdf/kr16_2_macro.xacro" />
-  <xacro:kuka_kr16_2 prefix="floor_" />
+<robot xmlns:xacro="http://www.ros.org/wiki/xacro" name="gantry">
+  <xacro:include filename="$(find kuka_kr16_support)/urdf/kr16_2_macro.xacro"/>
+  <xacro:kuka_kr16_2 prefix="floor_"/>
   <link name="root">
   </link>
   <joint name="root_floor" type="fixed">
-	  <origin xyz="0 1 0" rpy="0 0 0"/>
-	  <parent link="root" />
-	  <child link="floor_base_link" />
+    <origin xyz="0 1 0" rpy="0 0 0"/>
+    <parent link="root"/>
+    <child link="floor_base_link"/>
   </joint>
 </robot>

File: robotlab_support/urdf/gantry.xacro (robot description, xacro)
@@ -1,6 +1,6 @@
 <?xml version="1.0"?>
 <!--Generates a urdf from the macro in gantry_macro.xacro -->
-<robot name="gantry" xmlns:xacro="http://www.ros.org/wiki/xacro">
-  <xacro:include filename="$(find gantry_support)/urdf/gantry_robot_macro.xacro" />
+<robot xmlns:xacro="http://www.ros.org/wiki/xacro" name="gantry">
+  <xacro:include filename="$(find gantry_support)/urdf/gantry_robot_macro.xacro"/>
   <xacro:gantry_robot prefix="gantry_"/>
 </robot>

File: robotlab_support/urdf/robotlab.xacro (robot description, xacro)
@@ -1,6 +1,6 @@
 <?xml version="1.0"?>
 <!--Generates a urdf from the macro in gantry_macro.xacro -->
-<robot name="robotlab" xmlns:xacro="http://www.ros.org/wiki/xacro">
-	<xacro:include filename="$(find robotlab_support)/urdf/robotlab_macro.xacro" />
-	<xacro:robotlab prefix="" />
+<robot xmlns:xacro="http://www.ros.org/wiki/xacro" name="robotlab">
+  <xacro:include filename="$(find robotlab_support)/urdf/robotlab_macro.xacro"/>
+  <xacro:robotlab prefix=""/>
 </robot>
