Commit message: xmllint formatting

File: robotlab_support/urdf/robotlab_macro.xacro (robot description, xacro)
@@ -2,73 +2,73 @@
 <!--Generates a urdf from the macro in gantry_macro.xacro -->
 <robot xmlns:xacro="http://www.ros.org/wiki/xacro">
-	<xacro:macro name="robotlab" params="prefix">
-		<!-- Load required files -->
-		<xacro:include filename="$(find gantry_support)/urdf/gantry_robot_macro.xacro" />
-		<xacro:include filename="$(find kuka_kr16_support)/urdf/kr16_2_macro.xacro" />
-		<xacro:include filename="$(find robotlab_support)/urdf/schunk_macro.xacro" />
-		<xacro:include filename="$(find	robotlab_support)/urdf/utility_plate_macro.xacro" />
-		<!-- Run macros -->
-		<xacro:gantry_robot prefix="${prefix}gantry_" />
-		<xacro:kuka_kr16_2 prefix="${prefix}floor_" />
-		<xacro:FTC-50-80 prefix="${prefix}gantry_" />
-		<xacro:FTC-50-80 prefix="${prefix}floor_" />
-		<xacro:SWK-020 prefix="${prefix}gantry_" />
-		<xacro:SWK-020 prefix="${prefix}floor_" />
-		<xacro:A1_plate prefix="${prefix}gantry_" />
-		<xacro:A1_plate prefix="${prefix}floor_" />
-		<xacro:A3_box prefix="${prefix}floor_" />
-		<xacro:A3_box prefix="${prefix}gantry_" />
-		<link name="${prefix}root">
+  <xacro:macro name="robotlab" params="prefix">
+    <!-- Load required files -->
+    <xacro:include filename="$(find gantry_support)/urdf/gantry_robot_macro.xacro"/>
+    <xacro:include filename="$(find kuka_kr16_support)/urdf/kr16_2_macro.xacro"/>
+    <xacro:include filename="$(find robotlab_support)/urdf/schunk_macro.xacro"/>
+    <xacro:include filename="$(find robotlab_support)/urdf/utility_plate_macro.xacro"/>
+    <!-- Run macros -->
+    <xacro:gantry_robot prefix="${prefix}gantry_"/>
+    <xacro:kuka_kr16_2 prefix="${prefix}floor_"/>
+    <xacro:FTC-50-80 prefix="${prefix}gantry_"/>
+    <xacro:FTC-50-80 prefix="${prefix}floor_"/>
+    <xacro:SWK-020 prefix="${prefix}gantry_"/>
+    <xacro:SWK-020 prefix="${prefix}floor_"/>
+    <xacro:A1_plate prefix="${prefix}gantry_"/>
+    <xacro:A1_plate prefix="${prefix}floor_"/>
+    <xacro:A3_box prefix="${prefix}floor_"/>
+    <xacro:A3_box prefix="${prefix}gantry_"/>
+    <link name="${prefix}root">
 		</link>
-		<joint name="${prefix}root_gantry" type="fixed">
-			<origin xyz="0 0 0.0" rpy="0 0 0" />
-		        <parent link="${prefix}root" />
-		        <child link="${prefix}gantry_root" />
-		</joint>
-		<joint name="${prefix}root_floor" type="fixed">
-		        <origin xyz="-0.402 0.486 0" rpy="0 0 -${KUKA_DEG2RAD * 90}"/>
-		        <parent link="${prefix}root" />
-		        <child link="${prefix}floor_base_link" />
-		</joint>
-		<joint name="${prefix}gantry_tool0_ftc" type="fixed">
-			<origin xyz="0 0 0" rpy="0 0 0"/>
-			<parent link="${prefix}gantry_tool0" />
-			<child link="${prefix}gantry_FTC-50-80" />
-		</joint>
-		<joint name="${prefix}gantry_ftc_sws" type="fixed">
-			<origin xyz="0 0 0.0485" rpy="0 0 0"/>
-			<parent link="${prefix}gantry_FTC-50-80" />
-			<child link="${prefix}gantry_SWK-020" />
-		</joint>
-		<joint name="${prefix}floor_tool0_ftc" type="fixed">
-			<origin xyz="0 0 0" rpy="0 0 0"/>
-			<parent link="${prefix}floor_tool0" />
-			<child link="${prefix}floor_FTC-50-80" />
-		</joint>
-		<joint name="${prefix}floor_ftc_sws" type="fixed">
-			<origin xyz="0 0 0.0485" rpy="0 0 0"/>
-			<parent link="${prefix}floor_FTC-50-80" />
-			<child link="${prefix}floor_SWK-020" />
-		</joint>
-		<joint name="${prefix}gantry_A1_utility" type="fixed">
-			<origin xyz="0.1 0.30 -0.25" rpy="0 0 0" />
-			<parent link="${prefix}gantry_link_1" />
-			<child link="${prefix}gantry_A1_utility_plate" />
-		</joint>
-		<joint name="${prefix}floor_A1_utility" type="fixed">
-			<origin xyz="0.1 0.30 -0.25" rpy="0 0 0" />
-			<parent link="${prefix}floor_link_1" />
-			<child link="${prefix}floor_A1_utility_plate" />
-		</joint>
-		<joint name="${prefix}floor_A3_plate_box" type="fixed">
-			<origin xyz="-0.28 0.1 0.18" rpy="0 0 ${KUKA_DEG2RAD * 90}"/>
-			<parent link="${prefix}floor_link_3"/>
-			<child link="${prefix}floor_A3_box" />
-		</joint>
-		<joint name="${prefix}gantry_A3_plate_box" type="fixed">
-			<origin xyz="-0.28 0.1 0.18" rpy="0 0 ${KUKA_DEG2RAD * 90}"/>
-			<parent link="${prefix}gantry_link_3"/>
-			<child link="${prefix}gantry_A3_box" />
-		</joint>
-	</xacro:macro>
+    <joint name="${prefix}root_gantry" type="fixed">
+      <origin xyz="0 0 0.0" rpy="0 0 0"/>
+      <parent link="${prefix}root"/>
+      <child link="${prefix}gantry_root"/>
+    </joint>
+    <joint name="${prefix}root_floor" type="fixed">
+      <origin xyz="-0.402 0.486 0" rpy="0 0 -${KUKA_DEG2RAD * 90}"/>
+      <parent link="${prefix}root"/>
+      <child link="${prefix}floor_base_link"/>
+    </joint>
+    <joint name="${prefix}gantry_tool0_ftc" type="fixed">
+      <origin xyz="0 0 0" rpy="0 0 0"/>
+      <parent link="${prefix}gantry_tool0"/>
+      <child link="${prefix}gantry_FTC-50-80"/>
+    </joint>
+    <joint name="${prefix}gantry_ftc_sws" type="fixed">
+      <origin xyz="0 0 0.0485" rpy="0 0 0"/>
+      <parent link="${prefix}gantry_FTC-50-80"/>
+      <child link="${prefix}gantry_SWK-020"/>
+    </joint>
+    <joint name="${prefix}floor_tool0_ftc" type="fixed">
+      <origin xyz="0 0 0" rpy="0 0 0"/>
+      <parent link="${prefix}floor_tool0"/>
+      <child link="${prefix}floor_FTC-50-80"/>
+    </joint>
+    <joint name="${prefix}floor_ftc_sws" type="fixed">
+      <origin xyz="0 0 0.0485" rpy="0 0 0"/>
+      <parent link="${prefix}floor_FTC-50-80"/>
+      <child link="${prefix}floor_SWK-020"/>
+    </joint>
+    <joint name="${prefix}gantry_A1_utility" type="fixed">
+      <origin xyz="0.1 0.30 -0.25" rpy="0 0 0"/>
+      <parent link="${prefix}gantry_link_1"/>
+      <child link="${prefix}gantry_A1_utility_plate"/>
+    </joint>
+    <joint name="${prefix}floor_A1_utility" type="fixed">
+      <origin xyz="0.1 0.30 -0.25" rpy="0 0 0"/>
+      <parent link="${prefix}floor_link_1"/>
+      <child link="${prefix}floor_A1_utility_plate"/>
+    </joint>
+    <joint name="${prefix}floor_A3_plate_box" type="fixed">
+      <origin xyz="-0.28 0.1 0.18" rpy="0 0 ${KUKA_DEG2RAD * 90}"/>
+      <parent link="${prefix}floor_link_3"/>
+      <child link="${prefix}floor_A3_box"/>
+    </joint>
+    <joint name="${prefix}gantry_A3_plate_box" type="fixed">
+      <origin xyz="-0.28 0.1 0.18" rpy="0 0 ${KUKA_DEG2RAD * 90}"/>
+      <parent link="${prefix}gantry_link_3"/>
+      <child link="${prefix}gantry_A3_box"/>
+    </joint>
+  </xacro:macro>
 </robot>

File: robotlab_support/urdf/schunk_macro.xacro (robot description, xacro)
@@ -1,58 +1,58 @@
 <?xml version="1.0"?>
 <robot xmlns:xacro="http://www.ros.org/wiki/xacro">
-	<xacro:macro name="FTC-50-80" params="prefix">
-		<link name="${prefix}FTC-50-80" >
-    <visual>
-      <geometry>
-        <cylinder length="0.0485" radius="0.082"/>
-      </geometry>
-    </visual>
-    <collision>
-      <geometry>
-        <cylinder length="0.05" radius="0.1"/>
-      </geometry>
-    </collision>
-    <inertial>
-      <!-- data from http://www.comoso.com/uploads/showcase/manuals/Schunk_Comoso_eng_robot_accessoires.pdf -->
-      <mass value="1.56"/>
-      <inertia ixx="0.00395" ixy="0.0" ixz="0.0" iyy="0.00395" iyz="0.0" izz="0.0058"/>
-    </inertial>
-  </link>
-	</xacro:macro>
-	<xacro:macro name="SWA-020" params="prefix">
-		<link name="${prefix}SWA-020" >
-			<visual>
-	        		<origin xyz="0 0 0" rpy="0 0 0"/>
-	        		<geometry>
-			          	<mesh filename="package://robotlab_support/meshes/schunk/visual/SWA-020.stl" scale="0.001 0.001 0.001"/>
-        			</geometry>
-			      	</visual>
-    <inertial>
-      <!-- data from http://www.comoso.com/uploads/showcase/manuals/Schunk_Comoso_eng_robot_accessoires.pdf -->
-      <mass value="0.3"/>
-      <inertia ixx="0.054584" ixy="0.0" ixz="0.0" iyy="0.054584" iyz="0.0" izz="0.10914"/>
-    </inertial>
-		</link>
-	</xacro:macro>
-	<xacro:macro name="SWK-020" params="prefix">
-		<link name="${prefix}SWK-020" >
-			<visual>
-	        		<origin xyz="0 0 0" rpy="${pi/2} ${pi} 0"/>
-	        		<geometry>
-			          	<mesh filename="package://robotlab_support/meshes/schunk/visual/SWK-020.stl" scale="0.001 0.001 0.001"/>
-        			</geometry>
-			      	</visual>
-			<collision>
-	        		<origin xyz="0 0 0" rpy="${pi/2} ${pi} 0"/>
-	        		<geometry>
-			          	<mesh filename="package://robotlab_support/meshes/schunk/visual/SWK-020.stl" scale="0.002 0.002 0.002"/>
-        			</geometry>
-			      	</collision>
-    <inertial>
-      <!-- data from http://www.comoso.com/uploads/showcase/manuals/Schunk_Comoso_eng_robot_accessoires.pdf -->
-      <mass value="0.8"/>
-      <inertia ixx="0.14555" ixy="0.0" ixz="0.0" iyy="0.14555" iyz="0.0" izz="0.29104"/>
-    </inertial>
-		</link>
-	</xacro:macro>
+  <xacro:macro name="FTC-50-80" params="prefix">
+    <link name="${prefix}FTC-50-80">
+      <visual>
+        <geometry>
+          <cylinder length="0.0485" radius="0.082"/>
+        </geometry>
+      </visual>
+      <collision>
+        <geometry>
+          <cylinder length="0.05" radius="0.1"/>
+        </geometry>
+      </collision>
+      <inertial>
+        <!-- data from http://www.comoso.com/uploads/showcase/manuals/Schunk_Comoso_eng_robot_accessoires.pdf -->
+        <mass value="1.56"/>
+        <inertia ixx="0.00395" ixy="0.0" ixz="0.0" iyy="0.00395" iyz="0.0" izz="0.0058"/>
+      </inertial>
+    </link>
+  </xacro:macro>
+  <xacro:macro name="SWA-020" params="prefix">
+    <link name="${prefix}SWA-020">
+      <visual>
+        <origin xyz="0 0 0" rpy="0 0 0"/>
+        <geometry>
+          <mesh filename="package://robotlab_support/meshes/schunk/visual/SWA-020.stl" scale="0.001 0.001 0.001"/>
+        </geometry>
+      </visual>
+      <inertial>
+        <!-- data from http://www.comoso.com/uploads/showcase/manuals/Schunk_Comoso_eng_robot_accessoires.pdf -->
+        <mass value="0.3"/>
+        <inertia ixx="0.054584" ixy="0.0" ixz="0.0" iyy="0.054584" iyz="0.0" izz="0.10914"/>
+      </inertial>
+    </link>
+  </xacro:macro>
+  <xacro:macro name="SWK-020" params="prefix">
+    <link name="${prefix}SWK-020">
+      <visual>
+        <origin xyz="0 0 0" rpy="${pi/2} ${pi} 0"/>
+        <geometry>
+          <mesh filename="package://robotlab_support/meshes/schunk/visual/SWK-020.stl" scale="0.001 0.001 0.001"/>
+        </geometry>
+      </visual>
+      <collision>
+        <origin xyz="0 0 0" rpy="${pi/2} ${pi} 0"/>
+        <geometry>
+          <mesh filename="package://robotlab_support/meshes/schunk/visual/SWK-020.stl" scale="0.002 0.002 0.002"/>
+        </geometry>
+      </collision>
+      <inertial>
+        <!-- data from http://www.comoso.com/uploads/showcase/manuals/Schunk_Comoso_eng_robot_accessoires.pdf -->
+        <mass value="0.8"/>
+        <inertia ixx="0.14555" ixy="0.0" ixz="0.0" iyy="0.14555" iyz="0.0" izz="0.29104"/>
+      </inertial>
+    </link>
+  </xacro:macro>
 </robot>
