Commit message: Add origin to world-root joint

File: robotlab_gazebo/urdf/robotlab.xacro (robot description, xacro)
@@ -8,4 +8,5 @@
     <parent link="world"/>
     <child link="root"/>
+    <origin xyz="0.0 0.0 0.0" rpy="0.0 0.0 0.0" />
   </joint>
 </robot>

Commit message: Gravity fixes. Better colors for utility plates and equipment

File: robotlab_gazebo/urdf/robotlab.xacro (robot description, xacro)
@@ -8,5 +8,5 @@
     <parent link="world"/>
     <child link="root"/>
-    <origin xyz="0.0 0.0 0.0" rpy="0.0 0.0 0.0" />
+    <origin xyz="0.0 0.0 0.015" rpy="0.0 0.0 0.0" />
   </joint>
 </robot>

File: robotlab_gazebo/urdf/robotlab_macro.xacro (robot description, xacro)
@@ -1,4 +1,5 @@
 <?xml version="1.0"?>
-<robot xmlns:xacro="http://ros.org/wiki/xacro">
+<robot xmlns:xacro="http://www.ros.org/wiki/xacro">
+  <!-- Load needed macros -->
   <!-- Get the robotlab macro from support to generate the urdf of the robots -->
   <xacro:include filename="$(find robotlab_support)/urdf/robotlab_macro.xacro"/>
@@ -8,56 +9,30 @@
   <!-- Load gazebo_ros_control plugin -->
   <xacro:include filename="$(find robotlab_gazebo)/urdf/gazebo.xacro"/>
+  <!-- Load gravity config for gantry and KR16 -->
+  <xacro:include filename="$(find gantry_gazebo)/urdf/gantry_gravity_macro.xacro" />
+  <xacro:include filename="$(find kuka_kr16_gazebo)/urdf/kr16_2_gravity_macro.xacro" />
+  <!-- Load colors for utility plates -->
+  <xacro:include filename="$(find robotlab_gazebo)/urdf/utility_plate_gazebo_macro.xacro" />
+  <!-- Done loading macros -->
   <!-- Make the Gazebo version of the robotlab macro  -->
   <xacro:macro name="robotlab_gazebo" params="prefix" >
     <!-- load robots -->
     <xacro:robotlab prefix="${prefix}" />
-    <!-- load gantry transmission -->
+    <!-- Utility plate colors -->
+    <xacro:A1_plate_gazebo prefix="${prefix}gantry_" />
+    <xacro:A3_box_gazebo prefix="${prefix}gantry_" />
+    <xacro:A1_plate_gazebo prefix="${prefix}floor_" />
+    <xacro:A3_box_gazebo prefix="${prefix}floor_" />
+    <!-- load transmission files for gantry and KR16 -->
     <xacro:gantry_transmission prefix="${prefix}gantry_" />
-    <!-- load gantry kr16 transmission -->
     <xacro:kr16_2_transmission prefix="${prefix}gantry_" />
-    <!-- load floor kr16 transmission -->
     <xacro:kr16_2_transmission prefix="${prefix}floor_" />
-    <!-- The robots have gravity compensation (spring system? Or breaks?) -->
-    <gazebo reference="${prefix}gantry_base_link">
-      <turnGravityOff>true</turnGravityOff>
-    </gazebo>
-    <gazebo reference="${prefix}gantry_link_1">
-      <turnGravityOff>true</turnGravityOff>
-    </gazebo>
-    <gazebo reference="${prefix}gantry_link_2">
-      <turnGravityOff>true</turnGravityOff>
-    </gazebo>
-    <gazebo reference="${prefix}gantry_link_3">
-      <turnGravityOff>true</turnGravityOff>
-    </gazebo>
-    <gazebo reference="${prefix}gantry_link_4">
-      <turnGravityOff>true</turnGravityOff>
-    </gazebo>
-    <gazebo reference="${prefix}gantry_link_5">
-      <turnGravityOff>true</turnGravityOff>
-    </gazebo>
-    <gazebo reference="${prefix}gantry_link_6">
-      <turnGravityOff>true</turnGravityOff>
-    </gazebo>
-    <gazebo reference="${prefix}floor_base_link">
-      <turnGravityOff>true</turnGravityOff>
-    </gazebo>
-    <gazebo reference="${prefix}floor_link_1">
-      <turnGravityOff>true</turnGravityOff>
-    </gazebo>
-    <gazebo reference="${prefix}floor_link_2">
-    <turnGravityOff>true</turnGravityOff>
-    </gazebo>
-    <gazebo reference="${prefix}floor_link_3">
-      <turnGravityOff>true</turnGravityOff>
-    </gazebo>
-    <gazebo reference="${prefix}floor_link_4">
-      <turnGravityOff>true</turnGravityOff>
-    </gazebo>
-    <gazebo reference="${prefix}floor_link_5">
-      <turnGravityOff>true</turnGravityOff>
-    </gazebo>
-    <gazebo reference="${prefix}floor_link_6">
-      <turnGravityOff>true</turnGravityOff>
+    <!-- Load gravity settings -->
+    <!-- The robots only have position control. It compensates for gravity using servo and breaks -->
+    <xacro:gantry_gravity prefix="${prefix}gantry_" />
+    <xacro:kr16_2_gravity prefix="${prefix}gantry_" />
+    <xacro:kr16_2_gravity prefix="${prefix}floor_" />
+    <gazebo reference="${prefix}root">
+	<static>true</static>
     </gazebo>
     <!-- ros_control plugin loaded from kr_16 file-->

File: robotlab_support/urdf/robotlab_macro.xacro (robot description, xacro)
@@ -19,5 +19,6 @@
 		<link name="${prefix}root">
 		</link>
-		<joint name="${prefix}root_gantry_fixed" type="fixed">
+		<joint name="${prefix}root_gantry" type="fixed">
+			<origin xyz="0 0 0.0" rpy="0 0 0" />
 		        <parent link="${prefix}root" />
 		        <child link="${prefix}gantry_root" />
